File: PCB/DC_load/DC_load.sch (KiCad schematic (older format))
At the start: 2 parts

Commit message: prelimanary schematic
Parts:
- added C?: C_Small, Capacitors_SMD:C_0603, symbol Device:C_Small
- added C?: 1nF, Capacitors_SMD:C_0603, symbol Device:C_Small
- added C?: 100nF, Capacitors_SMD:C_0603, symbol Device:C_Small
- added D?: BAT54S, Package_TO_SOT_SMD:SOT-23, symbol Diode:BAT54S
- added HS?: Heatsink, symbol Mechanical:Heatsink
- added J?: Conn_01x02_Female, TerminalBlock_WAGO:TerminalBlock_WAGO-236_2Stift_RM5mm_2pol, symbol Connector:Conn_01x02_Female
- added J? (x2): Conn_01x02_Female, Connectors:Banana_Jack_2Pin, symbol Connector:Conn_01x02_Female
- added Q?: IRLB8721PBF, TO_SOT_Packages_THT:TO-220-3_Vertical, symbol Device:Q_NMOS_GDS
- added R? (x6): 2R2, Resistors_SMD:R_2512, symbol Device:R
- added R?: R_Small, Resistors_SMD:R_0603, symbol Device:R_Small
- added R?: 81k, Resistors_SMD:R_0603, symbol Device:R_Small
- added R? (x2): 10k, Resistors_SMD:R_0603, symbol Device:R_Small
- added R? (x2): 4k7, Resistors_SMD:R_0603, symbol Device:R_Small
- added TH?: NTCC-22K, Pin_Headers:Pin_Header_Straight_1x02_Pitch1.27mm, symbol Device:Thermistor_NTC
- added U?: MCP3421A1T-ECH, TO_SOT_Packages_SMD:SOT-23-6, symbol Analog_ADC:MCP3421A0T-ECH
- added U?: LMV321IDBVR, symbol Amplifier_Operational:LMV321
Connections:
- net labels added: +3V3, GND, NMOS_GATE, NTC_TEMP, PWM_MOS, SCL, SDA, V_MEAS
- wire segments 0 -> 95
Other:
- note added: "1mA (0.36mV) gives 2.88 counts\n1A (366.66mV) gives 2933,28 counts"
- note added: "30V input = 3.297V output"
- note added: "6x 2R2 = 0,366666667 mR\n@5A P= 9.16W (1.5W each)\n1mA current gives 360uV drop"
- note added: "@14bit res Vref=2.048V\n16383 counts\n1count = 0.125mV"
- note added: "MAX 5A"
- note added: "voltage follower\nfor mos gate control"

Commit message: schematic updated
Parts:
- added C2, C3: 100nF, Capacitors_SMD:C_0603, symbol Device:C_Small
- added J4: Conn_01x03, Connectors_JST:JST_EH_B03B-EH-A_03x2.50mm_Straight, symbol Connector_Generic:Conn_01x03
- added Q2: Q_NMOS_DGS, symbol Device:Q_NMOS_DGS
- added R11, R12, R13, R14: 10k, Resistors_SMD:R_0603, symbol Device:R_Small
- added U2, U3: LMV321IDBVR, Package_TO_SOT_SMD:SOT-23-5, symbol Amplifier_Operational:LMV321
- Q1: renamed from Q?; footprint TO_SOT_Packages_THT:TO-220-3_Vertical -> Package_TO_SOT_THT:TO-220-3_Vertical
- U1: renamed from U?; footprint (none) -> Package_TO_SOT_SMD:SOT-23-5
- U4: renamed from U?; footprint TO_SOT_Packages_SMD:SOT-23-6 -> Package_TO_SOT_SMD:SOT-23-6
- gave numbers to parts that had none: 23
Connections:
- net labels added: FAN_CONTROL, VCC
- wire segments 95 -> 133
Other:
- moved on the sheet: U4
